Commit message: Executes with 4 joints, still no gripper

File: lynxmotion/al5d.urdf (robot description, URDF)
Before this commit: robot al5d_arm, 8 links, 7 joints
Joints:
- joint base_joint: limit lower=-1.57 upper=1.57 effort=10 velocity=3 -> lower=-1.57 upper=1.57 effort=1 velocity=3
- joint elbow: limit lower=-1.57 upper=1.57 effort=10 velocity=3 -> lower=-1.57 upper=1.57 effort=1 velocity=3
- joint left_gripper: limit lower=-0.017 upper=0 effort=10 velocity=3 -> lower=-0.017 upper=0 effort=1 velocity=3; type fixed -> prismatic
- joint right_gripper: limit lower=-0.017 upper=0 effort=10 velocity=3 -> lower=0 upper=0.017 effort=1 velocity=3; type fixed -> prismatic
- joint shoulder_joint: limit lower=-1.553 upper=1.553 effort=0 velocity=3 -> lower=-1.553 upper=1.553 effort=1 velocity=3
- joint wrist: limit lower=-1.57 upper=1.57 effort=10 velocity=3 -> lower=-1.57 upper=1.57 effort=1 velocity=3
